Commit message: gazebo

File: src/my_robot_description/urdf/simple_robot.urdf (robot description, URDF)
Before this commit: robot simple_robot, 3 links, 2 joints
Links:
- link base_link: mass None -> 10.0; geometry collision box size=0.6 0.4 0.2; visual box size=0.6 0.4 0.2
- link left_wheel: mass None -> 1.0; geometry collision cylinder length=0.1 radius=0.1; visual cylinder length=0.1 radius=0.1
- link right_wheel: mass None -> 1.0; geometry collision cylinder length=0.1 radius=0.1; visual cylinder length=0.1 radius=0.1
